File: board/audio_out_pwm_stereo.kicad_sch (KiCad schematic)
At the start: 19 parts, among them U3 MCP6002-xP

Commit message: add title to schematics
Other:
- title: (none) -> https://github.com/Lougous/b68k-av
Changed lines of the file:
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@@
 (kicad_sch (version 20211123) (generator eeschema)
   (paper "A4")
+  (title_block
+    (title "https://github.com/Lougous/b68k-av")
+  )
   (junction (at 91.44 50.8) (diameter 0) (color 0 0 0 0)
   )
