File: board/av.kicad_sch (KiCad schematic)
At the start: 13 parts, among them J1 Conn_02x10_Odd_Even, J2 DB15_Female_HighDensity_Mount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, J8 Conn_01x05

Commit message: add title to schematics
Other:
- title: (none) -> https://github.com/Lougous/b68k-av
Changed lines of the file:
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@@
 (kicad_sch (version 20211123) (generator eeschema)
   (paper "A4")
+  (title_block
+    (title "https://github.com/Lougous/b68k-av")
+  )
   (junction (at 86.36 87.63) (diameter 0) (color 0 0 0 0)
   )
