File: board/bus_pld.kicad_sch (KiCad schematic)
At the start: 12 parts, among them J3 Conn_01x03, J5 Conn_02x05_Odd_Even, U1 74LS245, U2 EPM7064SL44

Commit message: add title to schematics
Other:
- title: (none) -> https://github.com/Lougous/b68k-av
Changed lines of the file:
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@@
 (kicad_sch (version 20211123) (generator eeschema)
   (paper "A4")
+  (title_block
+    (title "https://github.com/Lougous/b68k-av")
+  )
   (junction (at 113.03 34.29) (diameter 0) (color 0 0 0 0)
   )
