File: board/clocks.kicad_sch (KiCad schematic)
At the start: 4 parts, among them X1 CXO_DIP8, X3 CXO_DIP14

Commit message: add title to schematics
Other:
- title: (none) -> https://github.com/Lougous/b68k-av
Changed lines of the file:
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@@
 (kicad_sch (version 20211123) (generator eeschema)
   (paper "A4")
+  (title_block
+    (title "https://github.com/Lougous/b68k-av")
+  )
   (junction (at 86.36 25.4) (diameter 0) (color 0 0 0 0)
   )
