File: board/flex.kicad_sch (KiCad schematic)
At the start: 16 parts, among them J4 Conn_02x20_Odd_Even, J6 Conn_02x20_Odd_Even, U6 EPF10K10LC84, U7 74LS373, U8 74LS373

Commit message: add title to schematics
Other:
- title: (none) -> https://github.com/Lougous/b68k-av
Changed lines of the file:
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@@
 (kicad_sch (version 20211123) (generator eeschema)
   (paper "A4")
+  (title_block
+    (title "https://github.com/Lougous/b68k-av")
+  )
   (junction (at 90.17 82.55) (diameter 0) (color 0 0 0 0)
   )
