File: board/opl2.kicad_sch (KiCad schematic)
At the start: 2 parts, among them U11 YM3812

Commit message: add title to schematics
Other:
- title: (none) -> https://github.com/Lougous/b68k-av
Changed lines of the file:
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@@
 (kicad_sch (version 20211123) (generator eeschema)
   (paper "A4")
+  (title_block
+    (title "https://github.com/Lougous/b68k-av")
+  )
   (junction (at 119.38 83.82) (diameter 0) (color 0 0 0 0)
   )
