File: board/ramdac.kicad_sch (KiCad schematic)
At the start: 20 parts, among them U12 ADV476_DIP28, U4 LM337L_TO92

Commit message: add title to schematics
Other:
- title: (none) -> https://github.com/Lougous/b68k-av
Changed lines of the file:
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@@
 (kicad_sch (version 20211123) (generator eeschema)
   (paper "A4")
+  (title_block
+    (title "https://github.com/Lougous/b68k-av")
+  )
   (junction (at 196.85 64.77) (diameter 0) (color 0 0 0 0)
   )
